Commit message: Extend fer_bringup to real and MuJoCo as fer_ros2_bringup
- fer.urdf.xacro: upstream fer.urdf.xacro + one overlay via hardware:=real|mujoco
- controllers renamed to <interface>_<type>_controller; only broadcasters start active
- launch levels: fer_{real,mujoco}_ros2_control, fer_moveit, fer_moveit_skills,
  fer_moveit_skills_bt
- fix ros2_control deprecations (remap via spawner, antiwindup_strategy)
- add description-invariant test and CI

Co-Authored-By: Claude Opus 5

File: urdf/control/fer_real.ros2_control.xacro (robot description, xacro)
@@ -6,7 +6,6 @@
     Upstream franka_description's franka_arm.ros2_control.xacro targets the
     non-multi franka_hardware/FrankaHardwareInterface, which is NOT registered in
-    this workspace and uses a different param/interface contract. We suppress it
-    (ros2_control:=false on xacro:franka_robot in fer.xacro) and emit this instead.
-    See fer_ros2/TODO.md item 7.
+    this workspace and uses a different param/interface contract. fer.urdf.xacro
+    keeps it off (ros2_control:=false) and emits this instead for hardware:=real.
     Contract enforced by FrankaMultiHardwareInterface::on_init:
       hardware params : robot_count, ns<i>, robot_ip<i>   (i = 1 .. robot_count)
@@ -20,6 +19,6 @@
     they must NOT be declared here.
   -->
-  <xacro:macro name="fer_ros2_control" params="arm_id robot_ip">
-    <ros2_control name="${arm_id}_FrankaMultiHardwareInterface" type="system">
+  <xacro:macro name="fer_real_ros2_control" params="arm_id robot_ip">
+    <ros2_control name="${arm_id}_hardware" type="system">
       <hardware>
         <plugin>franka_hardware/FrankaMultiHardwareInterface</plugin>
